File: PCB/stepper-mouse-2025a/stepper-mouse-2025a.kicad_sch (KiCad schematic)
At the start: 84 parts, among them J1 STEPPER L, J2 STEPPER R, J3 Power, Q1 AO3401A, Q10 AO3402, Q11 BSS138, Q12 BSS138, Q13 BSS138, Q14 BSS138, Q2 AO3401A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

Commit message: Rev.1から使い勝手の悪いところを修正したもの
Connections:
- net +5VP: now also J1.1 (Pin_1), J2.1 (Pin_1); no longer J1.3 (Pin_3), J2.3 (Pin_3)
- net GND: now also R1.1, R2.2; no longer D1.1 (K), D2.1 (K)
- net LED1: now also D1.2 (A); no longer R1.2
- net LED2: now also D2.2 (A); no longer R2.1
- net STP1A renamed STP1P1
- net STP1P1: now also U1.27 (G16); no longer U1.29 (G5/SS)
- net STP1AX renamed STP1P1X
- net STP1B renamed STP1P2
- net STP1BX renamed STP1P2X
- net STP1P2X: now also J1.3 (Pin_3); no longer J1.4 (Pin_4)
- net STP1C renamed STP1P3
- net STP1P3: now also U1.29 (G5/SS); no longer U1.30 (G18/SCK)
- net STP1CX renamed STP1P3X
- net STP1P3X: now also J1.4 (Pin_4); no longer J1.1 (Pin_1)
- net STP1D renamed STP1P4
- net STP1P4: now also U1.30 (G18/SCK); no longer U1.27 (G16)
- net STP1DX renamed STP1P4X
- net STP2A renamed STP2P1
- net STP2P1: now also U1.7 (G32/ADC1_4); no longer U1.8 (G33/ADC1_5)
- net STP2AX renamed STP2P1X
- net STP2P1X: now also J2.2 (Pin_2); no longer J2.4 (Pin_4)
- net STP2B renamed STP2P2
- net STP2P2: now also U1.8 (G33/ADC1_5); no longer U1.9 (G25/ADC1_8)
- removed net STP2BX: D9.2 (A), J2.2 (Pin_2), Q8.3 (D)
- net STP2C renamed STP2P3
- net STP2P3: now also U1.9 (G25/ADC1_8); no longer U1.7 (G32/ADC1_4)
- removed net STP2CX: D8.2 (A), J2.5 (Pin_5), Q9.3 (D)
- net STP2D renamed STP2P4
- net STP2DX renamed STP2P4X
- net STP2P4X: now also J2.5 (Pin_5); no longer J2.1 (Pin_1)
- new net: D1.1 (K), R1.2
- new net: D2.1 (K), R2.1
- new net STP2P2X: D8.2 (A), J2.3 (Pin_3), Q8.3 (D)
- new net STP2P3X: D9.2 (A), J2.4 (Pin_4), Q9.3 (D)
Other:
- moved on the sheet: D1, D2, D8, D9, R1, R2

Commit message: Rev.2のエラッタを修正
Connections:
- net +5VP: now also J1.5 (Pin_5), J2.5 (Pin_5); no longer J1.1 (Pin_1), J2.1 (Pin_1)
- net STP1P1X: now also J1.4 (Pin_4); no longer J1.2 (Pin_2)
- net STP1P3X: now also J1.2 (Pin_2); no longer J1.4 (Pin_4)
- net STP1P4X: now also J1.1 (Pin_1); no longer J1.5 (Pin_5)
- net STP2P1X: now also J2.4 (Pin_4); no longer J2.2 (Pin_2)
- net STP2P3X: now also J2.2 (Pin_2); no longer J2.4 (Pin_4)
- net STP2P4X: now also J2.1 (Pin_1); no longer J2.5 (Pin_5)
Other:
- moved on the sheet: J1, J2
Changed lines of the file:
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@@
     )
   )
-  (symbol (lib_id "Connector_Generic:Conn_01x05") (at 267.97 93.98 0) (mirror y) (unit 1)
-    (in_bom yes) (on_board yes) (dnp no) (fields_autoplaced)
-    (property "Reference" "J2" (at 267.97 83.4857 0)
-      (effects (font (size 1.27 1.27)))
-    )
-    (property "Value" "STEPPER R" (at 267.97 85.9099 0)
+  (symbol (lib_id "Connector_Generic:Conn_01x05") (at 267.97 93.98 180) (unit 1)
+    (in_bom yes) (on_board yes) (dnp no)
+    (property "Reference" "J2" (at 267.97 104.4743 0)
+      (effects (font (size 1.27 1.27)))
+    )
+    (property "Value" "STEPPER R" (at 267.97 102.0501 0)
       (effects (font (size 1.27 1.27)))
     )
@@
     )
   )
-  (symbol (lib_id "Connector_Generic:Conn_01x05") (at 267.97 46.99 0) (mirror y) (unit 1)
-    (in_bom yes) (on_board yes) (dnp no) (fields_autoplaced)
-    (property "Reference" "J1" (at 267.97 36.4957 0)
-      (effects (font (size 1.27 1.27)))
-    )
-    (property "Value" "STEPPER L" (at 267.97 38.9199 0)
-      (effects (font (size 1.27 1.27)))
-    )
+  (symbol (lib_id "Connector_Generic:Conn_01x05") (at 267.97 46.99 180) (unit 1)
+    (in_bom yes) (on_board yes) (dnp no)
+    (property "Reference" "J1" (at 267.97 57.4843 0)
+      (effects (font (size 1.27 1.27)))
+    )
+    (property "Value" "STEPPER L" (at 267.97 55.0601 0)
+      (effects (font (size 1.27 1.27)))
+    )
